File: pcb/rev_2/amiga-1000-keyboard-rev2.kicad_pcb (KiCad board)
At the start: 2 copper layers, 389.2 x 145 mm, 235 parts, among them J1 AMIGA, J2 USB-C, J3 ISP, SW1 ESC, SW10 F9, SW11 F10, SW12 HELP, SW13 `, SW14 1, SW15 2, SW16 3, SW17 4, SW18 5, SW19 6, SW2 F1, SW20 7, SW21 8, SW22 9, SW23 0, SW24 -, SW25 =, SW26 \\, SW27 UP, SW28 TAB, SW29 Q, SW3 F2, SW30 W, SW31 E, SW32 R, SW33 T, SW34 Y, SW35 U, SW36 I, SW37 O, SW38 P, SW39 [, SW4 F3, SW40 ], SW41 RETURN, SW42 LEFT, SW43 CAPS LOCK, SW44 A, SW45 S, SW46 D, SW47 F, SW48 G, SW49 H, SW5 F4, SW50 J, SW51 K, SW52 L, SW53 ;, SW54 ', SW55 (RET) INTL, SW56 DEL, SW57 RIGHT, SW58 L SHIFT INTL, SW59 Z, SW6 F5, SW60 X, SW61 C, SW62 V, SW63 B, SW64 N, SW65 M, SW66 ,, SW67 ., SW68 /, SW69 SPACE, SW7 F6, SW70 BACKSPACE, SW71 DOWN, SW72 KP 9, SW73 KP 6, SW74 KP 3, SW75 KP ., SW76 KP 8, SW77 KP 5, SW78 KP 2, SW79 KP ENTER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

Commit message: move the rev 2 controller to the right and swap its buttons for jumper pads.
Parts:
- removed SW93: RESET, Button_Switch_SMD:SW_Push_1P1T_XKB_TS-1187A
- removed SW94: BOOT, Button_Switch_SMD:SW_Push_1P1T_XKB_TS-1187A
- added JP1: RESET, Jumper:SolderJumper-2_P1.3mm_Open_RoundedPad1.0x1.5mm, F.Cu at (266.0, 53.0)
- added JP2: BOOT, Jumper:SolderJumper-2_P1.3mm_Open_RoundedPad1.0x1.5mm, F.Cu at (276.0, 53.0)
- moved C8 108.0 mm to (310.6, 54.0)
- moved C1 108.0 mm to (295.0, 43.4)
- moved C2 108.0 mm to (304.0, 43.4)
- moved C3 108.0 mm to (296.5, 50.5)
- moved C4 108.0 mm to (303.5, 50.5)
- moved C5 108.0 mm to (307.0, 60.5)
- moved C6 108.0 mm to (313.0, 58.0)
- moved C7 108.0 mm to (287.0, 54.0)
- moved U1 108.0 mm to (300.0, 54.0)
- moved Y1 108.0 mm to (299.5, 43.4)
- moved C9 108.0 mm to (302.4, 64.4)
- moved R3 68.0 mm to (282.0, 60.0)
- moved R1 48.0 mm to (262.0, 49.0)
- moved R2 44.0 mm to (272.0, 49.0)
- moved TP1 22.0 mm to (238.0, 53.0)
Routing:
- net /KDAT: track 104.8 -> 223.7 mm, vias 4 -> 6
- net /AMIGA_PWR: track 41.8 -> 150.9 mm, vias 2 -> 0
- net /VBUS: track 76.1 -> 184.6 mm, vias 0 -> 1
- net /USB_DN_MCU: track 73.5 -> 181.5 mm
- net /USB_DP_MCU: track 72.2 -> 180.2 mm
- net /ROW3: track 328.4 -> 433.4 mm, vias 15 -> 17
- net /KCLK: track 123.6 -> 228.3 mm
- net +5V: track 161.5 -> 246.2 mm, vias 10 -> 16
- net /ROW6: track 370.8 -> 288.1 mm, vias 10 -> 9
- net /ROW7: track 404.8 -> 327.3 mm, vias 12 -> 10
- net /CAPS_LED_A: track 240.9 -> 311.0 mm, vias 4 -> 3
- net /COL11: track 271.6 -> 206.4 mm, vias 6 -> 8
- net /COL1: track 477.4 -> 541.9 mm, vias 8 -> 9
- net /COL5: track 520.9 -> 584.3 mm
- net /COL0: track 453.8 -> 512.9 mm, vias 4 -> 5
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
Commit message: add lcsc part numbers to rev 2, with 12 pf load caps for its 9 pf crystal.
Parts:
- C1, C2: value 22pF -> 12pF

Commit message: turn usb-c to the rear, clear of the amiga jack.
Parts:
- moved J2 17.7 mm to (140.0, 43.6), turned to 180 degrees
- moved U3 6.58 mm to (140.0, 53.0)
- moved R10 5.00 mm to (146.0, 53.5)
- moved R9 5.00 mm to (146.0, 50.0)
- moved R7 3.16 mm to (133.0, 51.0)
- moved R8 3.16 mm to (136.0, 51.0)
- moved F1 2.20 mm to (131.0, 44.0), turned to 90 degrees
Routing:
- net /ROW4: track 374.9 -> 467.4 mm
- net /RESET: track 79.7 -> 141.6 mm, vias 6 -> 4
- net /AMIGA_PWR: track 150.9 -> 195.8 mm, vias 0 -> 6
- net /USB_DP: track 51.0 -> 13.9 mm
- net /COL2: track 591.6 -> 563.8 mm, vias 12 -> 9
- net /COL3: track 619.5 -> 593.1 mm
- net /COL0: track 512.9 -> 490.3 mm, vias 5 -> 4
- net /USB_DN_MCU: track 181.5 -> 163.5 mm, vias 4 -> 0
- net /KDAT: track 223.7 -> 209.6 mm, vias 6 -> 2
- net /ROW0: track 324.6 -> 337.8 mm
- net /VBUS: track 184.6 -> 196.1 mm
- net /VCC_EXT: track 32.2 -> 21.5 mm, vias 3 -> 2
- net /ROW7: track 327.3 -> 337.9 mm, vias 10 -> 9
- net /COL11: track 206.4 -> 216.6 mm, vias 8 -> 6
- net /CC2: track 14.9 -> 4.76 mm
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